File: eagle/Mixer-01.sch (EAGLE design)
At the start: 58 parts, among them IC1 TL072P, IC2 TL072P, IC3 LM4558N

Commit message: Mixer-01.brd 結線を修正
Parts:
- C10: value 0.2u -> 0.1u
Changed lines of the file:
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@@
 <part name="C8" library="resistor" deviceset="C-EU" device="050-024X044" value="0.1u"/>
 <part name="C9" library="resistor" deviceset="C-EU" device="050-024X044" value="0.1u"/>
-<part name="C10" library="resistor" deviceset="C-EU" device="050-024X044" value="0.2u"/>
+<part name="C10" library="resistor" deviceset="C-EU" device="050-024X044" value="0.1u"/>
 <part name="C11" library="resistor" deviceset="C-EU" device="050-024X044" value="0.1u"/>
 <part name="C12" library="resistor" deviceset="C-EU" device="050-024X044" value="0.1u"/>

Commit message: Mixer-01.brd: 修正
Parts:
- C5, C6: device resistor:CPOL-EUE7.5-16 -> rcl:CPOL-EUE7.5-16
Changed lines of the file:
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@@
 <part name="P+3" library="supply1" deviceset="V+" device=""/>
 <part name="P-2" library="supply1" deviceset="V-" device=""/>
-<part name="C5" library="resistor" deviceset="CPOL-EU" device="E7.5-16" value="470u"/>
-<part name="C6" library="resistor" deviceset="CPOL-EU" device="E7.5-16" value="470u"/>
+<part name="C5" library="rcl" deviceset="CPOL-EU" device="E7.5-16" value="470u"/>
+<part name="C6" library="rcl" deviceset="CPOL-EU" device="E7.5-16" value="470u"/>
 <part name="C7" library="resistor" deviceset="C-EU" device="050-024X044" value="0.1u"/>
 <part name="C8" library="resistor" deviceset="C-EU" device="050-024X044" value="0.1u"/>

Commit message: 電池ボックスのGNDの配線を変更
Parts:
- added JP17: PWR-GND, pinhead:PINHD-1X1
Changed lines of the file:
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@@
 <part name="GND10" library="supply1" deviceset="GND" device=""/>
 <part name="JP16" library="pinhead" deviceset="PINHD-1X3" device="" value="VOL-R"/>
+<part name="JP17" library="pinhead" deviceset="PINHD-1X1" device="" value="PWR-GND"/>
+<part name="GND11" library="supply1" deviceset="GND" device=""/>
 </parts>
 <sheets>
@@
 <attribute name="VALUE" x="139.7" y="43.18" size="1.778" layer="96"/>
 </instance>
+<instance part="JP17" gate="G$1" x="106.68" y="162.56"/>
+<instance part="GND11" gate="1" x="116.84" y="160.02"/>
 </instances>
 <busses>
@@
 <wire x1="93.98" y1="25.4" x2="93.98" y2="27.94" width="0.1524" layer="91"/>
 </segment>
+<segment>
+<pinref part="GND11" gate="1" pin="GND"/>
+<wire x1="106.68" y1="162.56" x2="116.84" y2="162.56" width="0.1524" layer="91"/>
+</segment>
 </net>

Commit message: OPAMPの入力を接地
Parts:
- added R24, R25, R26, R27, R28, R29, R30, R31: 100k, rcl:R-EU_0207/7
Connections:
- net GND: now also R24.1, R25.1, R26.1, R27.1, R28.1, R29.1, R30.1, R31.1
- net N$10: now also R25.2
- net N$11: now also R26.2
- net N$12: now also R27.2
- net N$18: now also R30.2
- net N$23: now also R31.2
- net N$7: now also R28.2
- net N$8: now also R29.2
- net N$9: now also R24.2
Other:
- moved on the sheet: C1, C13, C14, C15, C16, C2, C3, C4, JP1, JP11, JP12, JP13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

Commit message: Mixer基板設計図にV-GND用ピンを追加
Parts:
- added JP18: V-GND, pinhead:PINHD-1X1
Changed lines of the file:
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@@
 <part name="GND18" library="supply1" deviceset="GND" device=""/>
 <part name="GND19" library="supply1" deviceset="GND" device=""/>
+<part name="JP18" library="pinhead" deviceset="PINHD-1X1" device="" value="V-GND"/>
+<part name="GND20" library="supply1" deviceset="GND" device=""/>
 </parts>
 <sheets>
@@
 <instance part="GND18" gate="1" x="38.1" y="22.86"/>
 <instance part="GND19" gate="1" x="38.1" y="2.54"/>
+<instance part="JP18" gate="G$1" x="81.28" y="162.56"/>
+<instance part="GND20" gate="1" x="91.44" y="160.02"/>
 </instances>
 <busses>
@@
 <pinref part="GND19" gate="1" pin="GND"/>
 </segment>
+<segment>
+<pinref part="GND20" gate="1" pin="GND"/>
+<wire x1="81.28" y1="162.56" x2="91.44" y2="162.56" width="0.1524" layer="91"/>
+</segment>
 </net>
